File: ilr-lm317_r1/ilr-lm317_r1.sch (KiCad schematic (older format))
At the start: 34 parts, among them U1 LM317_3PinPackage, U2 LM317_3PinPackage, U3 LM317_3PinPackage, U4 LM317_3PinPackage

Commit message: sync
Signed-off-by: John McMaster <johndmcmaster@gmail.com>
Parts:
- added J1: Barrel_Jack, footprint:DCJack(EJ508A-ND)2, symbol Barrel_Jack
- added R10, R12, R6, R8: NOLOAD, Resistors_SMD:R_0603, symbol R
- added R11, R13, R7, R9: 0, Resistors_SMD:R_0603, symbol R
- D1: footprint (none) -> LEDs:LED_0603
- D10, D11, D12, D13, D14, D15, D16, D17, D18, D19, D2, D20, D21, D22, D23, D24, D25, D3, D4, D5, D6, D7, D8, D9: footprint (none) -> LEDs:LED_D5.0mm
- R1: value R -> 442; footprint (none) -> Resistors_SMD:R_0603
- R2, R3, R4, R5: footprint (none) -> Resistors_THT:R_Axial_DIN0207_L6.3mm_D2.5mm_P10.16mm_Horizontal
- U1, U2, U3, U4: footprint (none) -> TO_SOT_Packages_SMD:TO-252-2
Connections:
- net GND: now also J1.2, J1.3, R11.2, R13.2, R7.2, R9.2; no longer D13.1 (K), D19.1 (K), D25.1 (K), D7.1 (K)
- net VCC: now also J1.1, R6.1
- net at D2.2 (A), R2.1, U1.1 (ADJ): now also R6.2
- net at D8.2 (A), R3.1, U2.1 (ADJ): now also R8.2
- net at D14.2 (A), R4.1, U3.1 (ADJ): now also R10.2
- net at D20.2 (A), R5.1, U4.1 (ADJ): now also R12.2
- new net: D7.1 (K), R7.1, R8.1
- new net: D13.1 (K), R10.1, R9.1
- new net: D19.1 (K), R11.1, R12.1
- new net: D25.1 (K), R13.1
Other:
- note added: "LM317\nCurrent mode pg 12: http://www.ti.com/lit/ds/symlink/lm317.pdf\nOr: http://www.bristolwatch.com/ccs/LM317.htm\nVdrop max: 1.3 V\n\n# LEDs\nVdropMin: 1.7V\nMax LEDs per string: (12 - 1.7) / 1.4 = 7.4\nGCD vs 24 is 6\n\nR selection\nIout = 1.25 / R\nR = 1.25 / 0.1 = 12.5\nChoose 13 as closest standard value\nI = 1.25 / 13 = 96 mA\nR power: I^2 * R = 0.096^2 * 13 = 0.12 W\nVdrop: 13 * 0.096 =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"
- note added: "ON indicator LED\nOther LEDs are invisible\nbut hazardous to eyes\n\nWL-SMCW blue LED\n20 mA listed in DS as typ drive\nVdrop typ 3.2 V, max 3.5 V\n(12 - 3.2) / 0.02 = 440 R\nClosest resistor: 442 R"
- note removed: "LM317\n\n# LEDs\nVdropMin: 1.7V\nMax LEDs per string: (12 - 1.7) / 1.4 = 7.4\nGCD vs 24 is 6\n\nR selection\nIout = 1.25 / R\nR = 1.25 / 0.1 = 12.5\nChoose 13 as closest standard value\nI = 1.25 / 13 = 96 mA\nR power: I^2 * R = 0.096^2 * 13 = 0.12 W"
- note removed: "ON indicator LED\nOther LEDs are invisible\nbut hazardous to eyes"
